File: pcb/Verifypad.kicad_pcb (KiCad board)
At the start: 2 copper layers, 49 x 51.5 mm, 11 parts, among them J1 Conn_01x04, SW1 SW_Push, SW2 SW_Push, U1 MOUDLE-SEEEDUINO-XIAO

Commit message: final final final pcb
Parts:
- SW1, SW2: footprint PCM_Switch_Keyboard_Cherry_MX:SW_Cherry_MX_PCB_1.00u -> Button_Switch_Keyboard:SW_Cherry_MX_1.00u_PCB
- moved SW2 2.87 mm to (197.0, 81.9)
- moved SW1 2.66 mm to (176.5, 81.9)
Routing:
- net GND: track 52.8 -> 60.8 mm
- net Net-(U1-PA5_A9_D9_MISO): track 26.4 -> 24.5 mm
- net Net-(U1-PA7_A8_D8_SCK): track 25.7 -> 24.5 mm
