File: pcb/Verifypad.kicad_sch (KiCad schematic)
At the start: 4 parts, among them J1 Conn_01x04, SW1 SW_Push, SW2 SW_Push, U1 MOUDLE-SEEEDUINO-XIAO

Commit message: final final final pcb
Parts:
- SW1, SW2: footprint PCM_marbastlib-choc:SW_choc_v1_1u -> Button_Switch_Keyboard:SW_Cherry_MX_1.00u_PCB
Changed lines of the file:
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@@
 			)
 		)
-		(property "Footprint" "PCM_marbastlib-choc:SW_choc_v1_1u"
+		(property "Footprint" "Button_Switch_Keyboard:SW_Cherry_MX_1.00u_PCB"
 			(at 99.06 72.39 0)
 			(hide yes)
@@
 			)
 		)
-		(property "Footprint" "PCM_marbastlib-choc:SW_choc_v1_1u"
+		(property "Footprint" "Button_Switch_Keyboard:SW_Cherry_MX_1.00u_PCB"
 			(at 99.06 62.23 0)
 			(hide yes)
